File: PCB/Teclado3Teclas.kicad_pcb (KiCad board)
At the start: 2 copper layers, 67.9 x 47.1 mm, 8 parts, among them J1 Conn_01x04_Pin, SW1 SW_Push, SW2 SW_Push, SW3 SW_Push, U1 MOUDLE-SEEEDUINO-XIAO

Commit message: Add files via upload
Parts:
- moved D3 9.66 mm to (181.1, 119.0), turned to -90 degrees
- moved D2 9.51 mm to (161.9, 119.8), turned to -90 degrees
- moved D1 9.35 mm to (142.7, 119.1), turned to -90 degrees
Routing:
- net Net-(D2-DOUT): track 18.6 -> 49.5 mm, vias 2 -> 0
- net Net-(U1-PA10_A2_D2): track 41.4 -> 70.8 mm, vias 1 -> 0
- net +3V3: track 108.9 -> 126.2 mm, vias 1 -> 3
- net Net-(D1-DOUT): track 19.5 -> 31.4 mm
- net Net-(D1-DIN): track 28.5 -> 37.2 mm, vias 0 -> 1
- net Net-(U1-PA02_A0_D0): track 38.6 -> 42.5 mm
- net GND: track 114.1 -> 113.4 mm, vias 6 -> 0
